Commit message: Atualiza modelo do ator e adiciona novos objetos ao mundo de simulação

File: src/p3at_simulation/urdf/actor.xacro (robot description, xacro)
@@ -5,5 +5,5 @@
       <origin xyz="0 0 0" />
       <mass value="1.0" />
-      <inertia  ixx="1.0" ixy="0.0"  ixz="0.0"  iyy="100.0"  iyz="0.0"  izz="1.0" />
+      <inertia  ixx="3.0" ixy="0.0"  ixz="0.0"  iyy="100.0"  iyz="0.0"  izz="4.0" />
     </inertial>
     <visual>
